Commit message: añadir modelo de colisiones

File: ejercicio1/ej1.urdf (robot description, URDF)
Before this commit: robot ej1, 3 links, 2 joints
Links:
- link base_link: mass None -> 10.0; geometry collision box size=1 1 0.5; visual box size=1 1 0.5
- link horizontal_link: mass None -> 1.0; geometry collision box size=0.3 1.5 0.3; visual box size=0.3 1.5 0.3
- link vertical_link: mass None -> 1.0; geometry collision box size=0.3 0.3 2.5; visual box size=0.3 0.3 2.5
Joints:
- joint base2vertical: origin xyz=0 0 0.025 rpy=0 0 0 -> xyz=0 0 0.25 rpy=0 0 0
- joint vertical2horizontal: origin xyz=0 0 0.4 rpy=0 0 0 -> xyz=0 0 2.5 rpy=0 0 0

Commit message: arreglar dimensiones

File: ejercicio1/ej1.urdf (robot description, URDF)
Before this commit: robot ej1, 3 links, 2 joints
Links:
- link horizontal_link: geometry collision box size=0.3 1 0.3; visual box size=0.3 1 0.3
- link vertical_link: geometry collision box size=0.3 0.3 2; visual box size=0.3 0.3 2
